File: pcb/gate_sensor_v2.kicad_pcb (KiCad board)
At the start: 2 copper layers, 75 x 66 mm, 14 parts, among them J2 PWR_IN_ScrewTerm, J4 PWR_SW_JST_PH_2pin, U1 Arduino_Nano_Socket, U2 RXB6_433MHz_DirectSolder, U3 Heltec_LoRa32_V3

Commit message: Adjust silkscreen labels: center socket names, add USB label to Nano
- Move Heltec/Nano/RXB6 socket labels up for better vertical centering
- Add "USB" label at top of Arduino Nano socket frame
- Center R1 2k2 label above resistor body
Other:
- board text added: "USB"
Changed lines of the file:
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@@
   (gr_text "U3  HELTEC LoRa32 V3" (at 16.0000 6.0000) (layer "F.Fab")
     (effects (font (size 0.8000 0.8000) (thickness 0.1500))))
-  (gr_text "HELTEC LoRa32 V3" (at 17.4300 39.3400 90.0000) (layer "F.SilkS")
+  (gr_text "HELTEC LoRa32 V3" (at 17.4300 34.3400 90.0000) (layer "F.SilkS")
     (effects (font (size 0.8000 0.8000) (thickness 0.1500))))
-  (gr_text "SOCKET" (at 19.9300 35.3400 90.0000) (layer "F.SilkS")
+  (gr_text "SOCKET" (at 19.9300 30.3400 90.0000) (layer "F.SilkS")
     (effects (font (size 0.8000 0.8000) (thickness 0.1500))))
   (gr_text "GND" (at 2.0000 9.6700) (layer "F.SilkS")
@@
   (gr_text "U1  ARDUINO NANO" (at 55.0000 8.0000) (layer "F.Fab")
     (effects (font (size 0.8000 0.8000) (thickness 0.1500))))
-  (gr_text "ARDUINO NANO" (at 61.6200 35.7800 90.0000) (layer "F.SilkS")
+  (gr_text "ARDUINO NANO" (at 61.6200 30.7800 90.0000) (layer "F.SilkS")
     (effects (font (size 0.8000 0.8000) (thickness 0.1500))))
-  (gr_text "SOCKET" (at 64.1200 33.7800 90.0000) (layer "F.SilkS")
+  (gr_text "SOCKET" (at 64.1200 28.7800 90.0000) (layer "F.SilkS")
+    (effects (font (size 0.8000 0.8000) (thickness 0.1500))))
+  (gr_text "USB" (at 62.6200 12.5000) (layer "F.SilkS")
     (effects (font (size 0.8000 0.8000) (thickness 0.1500))))
   (gr_text "D13" (at 51.5000 11.6700) (layer "F.SilkS")
@@
   (gr_text "U2 RXB6 433MHz" (at 43.0000 9.0000) (layer "F.Fab")
     (effects (font (size 0.8000 0.8000) (thickness 0.1500))))
-  (gr_text "RXB6 433MHz" (at 44.0000 37.3200 90.0000) (layer "F.SilkS")
+  (gr_text "RXB6 433MHz" (at 44.0000 32.3200 90.0000) (layer "F.SilkS")
     (effects (font (size 0.8000 0.8000) (thickness 0.1500))))
   (gr_text "DIRECT SOLDER" (at 42.0000 55.6400) (layer "F.Fab")
@@
   (gr_line (start 42.2000 26.1000) (end 34.7200 26.1000) (layer "F.Fab") (width 0.1000))
   (gr_line (start 34.7200 26.1000) (end 34.7200 23.3000) (layer "F.Fab") (width 0.1000))
-  (gr_text "R1 2k2" (at 35.9200 21.2000) (layer "F.SilkS")
+  (gr_text "R1 2k2" (at 38.4600 21.7000) (layer "F.SilkS")
     (effects (font (size 0.8000 0.8000) (thickness 0.1500))))
   (gr_line (start 34.5200 24.8000) (end 37.3200 24.8000) (layer "F.Fab") (width 0.1000))
