File: pcb/gate_sensor_v2_assembly.kicad_pcb (KiCad board)
At the start: 2 copper layers, 75 x 66 mm, 14 parts, among them J2 PWR_IN_ScrewTerm, J4 PWR_SW_JST_PH_2pin, U1 Arduino_Nano_Socket, U2 RXB6_433MHz_DirectSolder, U3 Heltec_LoRa32_V3

Commit message: Adjust silkscreen labels: center socket names, add USB label to Nano
- Move Heltec/Nano/RXB6 socket labels up for better vertical centering
- Add "USB" label at top of Arduino Nano socket frame
- Center R1 2k2 label above resistor body
Other:
- board text added: "USB"
Changed lines of the file:
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@@
   (gr_text "U3  HELTEC LoRa32 V3" (at 16.0000 6.0000) (layer "F.Fab")
     (effects (font (size 0.8000 0.8000) (thickness 0.1500))))
-  (gr_text "HELTEC LoRa32 V3" (at 17.4300 39.3400 90.0000) (layer "F.SilkS")
+  (gr_text "HELTEC LoRa32 V3" (at 17.4300 34.3400 90.0000) (layer "F.SilkS")
     (effects (font (size 0.8000 0.8000) (thickness 0.1500))))
-  (gr_text "SOCKET" (at 19.9300 35.3400 90.0000) (layer "F.SilkS")
+  (gr_text "SOCKET" (at 19.9300 30.3400 90.0000) (layer "F.SilkS")
     (effects (font (size 0.8000 0.8000) (thickness 0.1500))))
   (gr_text "GND" (at 2.0000 9.6700) (layer "F.SilkS")
@@
   (gr_text "U1  ARDUINO NANO" (at 55.0000 8.0000) (layer "F.Fab")
     (effects (font (size 0.8000 0.8000) (thickness 0.1500))))
-  (gr_text "ARDUINO NANO" (at 61.6200 35.7800 90.0000) (layer "F.SilkS")
+  (gr_text "ARDUINO NANO" (at 61.6200 30.7800 90.0000) (layer "F.SilkS")
     (effects (font (size 0.8000 0.8000) (thickness 0.1500))))
-  (gr_text "SOCKET" (at 64.1200 33.7800 90.0000) (layer "F.SilkS")
+  (gr_text "SOCKET" (at 64.1200 28.7800 90.0000) (layer "F.SilkS")
+    (effects (font (size 0.8000 0.8000) (thickness 0.1500))))
+  (gr_text "USB" (at 62.6200 12.5000) (layer "F.SilkS")
     (effects (font (size 0.8000 0.8000) (thickness 0.1500))))
   (gr_text "D13" (at 51.5000 11.6700) (layer "F.SilkS")
@@
   (gr_text "U2 RXB6 433MHz" (at 43.0000 9.0000) (layer "F.Fab")
     (effects (font (size 0.8000 0.8000) (thickness 0.1500))))
-  (gr_text "RXB6 433MHz" (at 44.0000 37.3200 90.0000) (layer "F.SilkS")
+  (gr_text "RXB6 433MHz" (at 44.0000 32.3200 90.0000) (layer "F.SilkS")
     (effects (font (size 0.8000 0.8000) (thickness 0.1500))))
   (gr_text "DIRECT SOLDER" (at 42.0000 55.6400) (layer "F.Fab")
@@
   (gr_line (start 42.2000 26.1000) (end 34.7200 26.1000) (layer "F.Fab") (width 0.1000))
   (gr_line (start 34.7200 26.1000) (end 34.7200 23.3000) (layer "F.Fab") (width 0.1000))
-  (gr_text "R1 2k2" (at 35.9200 21.2000) (layer "F.SilkS")
+  (gr_text "R1 2k2" (at 38.4600 21.7000) (layer "F.SilkS")
     (effects (font (size 0.8000 0.8000) (thickness 0.1500))))
   (gr_line (start 34.5200 24.8000) (end 37.3200 24.8000) (layer "F.Fab") (width 0.1000))

Commit message: PCB v2.4: add Heltec GPIO48 -> R6 -> Nano D4 RX path
Enables bidirectional UART between the Heltec LoRa32 V3 and the Arduino
Nano. The Nano can now receive Meshtastic serial frames in addition to
sending RF events on D3.

R6 (4.7k) sits in series on the new trace as a back-feed limiter: when
the Heltec is USB-powered alone (e.g. during flashing) and the Nano's
5V rail is off, GPIO48 driving HIGH would otherwise forward-bias the
Nano's ESD clamp diodes into an unpowered Vcc rail. 4.7k caps the
current at ~0.57 mA, well below the clamp-diode rating.

PCB:
  - New nets HELTEC_TX and D4, R6 footprint at (48-53.08, 8.7)
  - HELTEC_TX routed F.Cu east through R14/R15 gap, B.Cu vertical at
    X=34 past the HELTEC_RX horizontal, F.Cu along top margin (Y=8.7)
    to R6 pad1
  - D4 routed F.Cu along Y=8.7 to X=73, via to B.Cu, right-edge drop
    to Nano R9
  - Removed redundant "75x66mm 2L 1.6mm HASL" subtitle to free silk
    space for the R6 label above the resistor
  - Enlarged bottom branding text from 0.7 to 1.0 mm
  - J4 bottom label "IN OUT" -> "Switch"
  - R6 added to assembly PCB 3D model list
  - 0 DRC violations, 40/40 netlist self-tests pass

Firmware:
  - config.h SERIAL_RX comment updated to reflect the real RX path
  - No code changes: firmware still only writes on D3 for now

Makefile:
  - New `make open` and `make open-assembly` targets that launch the
    board in the local KiCad AppImage

Docs:
  - Schematic ASCII diagram, netlist table, and hardening-components
    table updated for the new signal path and R6
  - pcb.md v2.4 changelog section added
  - bom.md adds R6 entry
  - firmware.md pin map updated
Parts:
- added R6: 4.7k, R6, F.Cu at (50.5, 8.70)
Connections:
- U1 pad R9: (no net) -> D4
- U3 pad L14: (no net) -> HELTEC_TX
Routing:
- net HELTEC_TX: track 0.00 -> 77.9 mm, vias 0 -> 2
- net D4: track 0.00 -> 46.3 mm, vias 0 -> 1
Other:
- board text added: "GATE SENSOR CARRIER v2.4"
- board text added: "GPIO48 series"
- board text added: "LOGIC LEVEL: D3->R1(2k2)->R2(3k3)->GND, jct->GPIO47; GPIO48->R6(4k7)->D4"
- board text added: "R6 4k7"
- board text added: "Switch"
- board text removed: "75x66mm 2L 1.6mm HASL"
- board text removed: "GATE SENSOR CARRIER v2.3"
- board text removed: "IN OUT"
- board text removed: "LOGIC LEVEL: D3->R1(2k2)->R2(3k3)->GND, jct->GPIO47"
